Commit message: lidar test implemented. ready for Pi

File: src/buildon_main/urdf/olaf.urdf (robot description, URDF)
Before this commit: robot olaf, 5 links, 4 joints
Links:
- removed link left_back_wheel
- removed link right_back_wheel
- added link axis_link, mass 0.10; collision box size=0.01 0.01 0.02; visual box size=0.01 0.01 0.02
- added link back_wheel, mass 0.1; collision cylinder length=0.01 radius=0.02; visual cylinder length=0.01 radius=0.02
- added link lidar_link, mass 0.05; collision cylinder length=0.04 radius=0.05; visual cylinder length=0.04 radius=0.05
- link base_link: mass 10.0 -> 5.0
Joints:
- removed joint left_back_wheel_joint
- removed joint right_back_wheel_joint
- added joint axis_joint: type continuous, parent base_link, child axis_link, origin xyz=-0.2 0 -0.11 rpy=0.0 0.0 0.0, axis 0.0 0 1
- added joint back_wheel_joint: type continuous, parent axis_link, child back_wheel, origin xyz=-0.01 0 0 rpy=0.0 0.0 0.0, axis 0.0 1 0
- added joint rostopic: type fixed, parent base_link, child lidar_link, origin xyz=0.0 0.0 0.12 rpy=0.0 0.0 0.0

File: src/buildon_main/urdf/olaf_copy.urdf (robot description, URDF)
Before this commit: robot olaf, 5 links, 4 joints
Links:
- added link lidar_link, mass 0.05; collision cylinder length=0.04 radius=0.05; visual cylinder length=0.04 radius=0.05
- added link right_wheel2, mass 1.0; collision cylinder length=0.05 radius=0.08; visual cylinder length=0.05 radius=0.08
- link axis_link: mass 10.0 -> 0.10
- link back_wheel: mass 1.0 -> 0.1
- link base_link: mass 10.0 -> 5.0
Joints:
- added joint lidar_joint: type fixed, parent base_link, child lidar_link, origin xyz=0.0 0.0 0.12 rpy=0.0 0.0 0.0
- added joint right_wheel_joint2: type fixed, parent base_link, child right_wheel2, origin xyz=0.3 -0.25 -0.05 rpy=0.0 0.0 0.0, axis 0.0 1 0
